File: hardware/kicad/dpaa_dist/dpaa_dist.kicad_sch (KiCad schematic)
At the start: 206 parts, among them J1 2x6, J10 2x6, J11 2x6, J12 2x6, J13 2x6, J14 2x6, J15 2x6, J16 2x6, J17 RJ45, J18 5.5/2.1, J2 2x6, J20 IDC 2x15, J21 IDC 2x15, J25 ESP32, J26 3.5mm, J27 3.5mm, J3 2x6, J4 2x6, J5 2x6, J6 2x6, J7 2x6, J8 2x6, J9 2x6, Q1 AO4407A, SW1 кнопка, U1 74LVC244A, U10 74LVC244A, U11 74LVC244A, U12 74LVC244A, U13 74LVC244A, U2 74LVC244A, U20 AP2112K-3.3, U21 AP2112K-3.3, U3 74LVC244A, U31 PCM5102A, U32 TDA1308, U4 74LVC244A, U5 74LVC244A, U6 74LVC244A, U7 74LVC244A, U8 74LVC244A, U9 74LVC244A

Commit message: Распределительная плата: порт Ethernet (P1 -> MagJack), плата 100x180, исправлена нумерация вилок IDC
- J19 = гребёнка P1 платы расширения (третий прямой шлейф IDC 2x15), J29 = RJ45 MagJack
  UDE RB1-125B8G1A (1000BASE-T, трансформаторы и терминация Боба Смита внутри, общий вывод
  и экран — на отдельную цепь CHASSIS: полигон под гнездом на обоих слоях, к земле через
  C306 1 нФ 2 кВ || R306 1 МОм); центральный отвод — C301 100 нФ, R301 0 Ом (DNP) к 3,3 В.
- Пары MDI разведены вручную одним слоем каждая (пары 1, 2 — верх, 3, 4 — низ), 45°, без
  переходных, сплошная земля другого слоя под ними, прочие цепи не ближе 1 мм; пары 2 и 4 —
  с обратной полярностью (без пересечений; PHY исправляет полярность). Расчёт волнового
  сопротивления и длины линий — README, gen/eth_lengths.txt.
- Исправлено: контакты вилок J20/J21 (и J19) теперь назначены с учётом зигзаг-нумерации
  футпринта IDC против нумерации 1-15/16-30 гребёнок платы расширения (прямой шлейф
  соединяет по положению); раньше сигналы стояли на чужих контактах.
- Плата 100x180: краевые разъёмы сдвинуты вниз, шина +5 В обходит MagJack по краю и ныряет
  под VIN через переходные; силовые C10/C11 переименованы в C101/C102 (дублировали C10/C11
  буферов); переходные земли у каждого конденсатора развязки; земля вилок через заливку
  (запрет вертикали между рядами J20/J21), автосшивка кусков земли (gen/stitch_fix.py).
- DRC: 0 ошибок, 0 неподключённых (4 предупреждения: концы шин 5V_B/5V_D, узкие перешейки
  заливки); ERC 0. Пакет fab/ перегенерирован; BOM: J29 C363353, C306 C135917, R301 исключён.
- Документация: README (раздел Ethernet, нумерация шлейфов), purchase.md (3 шлейфа, MagJack),
  wiring.md (W3, W29), bom.csv, schematics.md.

Co-Authored-By: Claude Fable 5.1 <noreply@anthropic.com>
Parts:
- removed C10: 1000u, CP_Radial_D10.0mm_P5.00mm, symbol dpaa:1000u_2
- removed C11: 10u, C_0805_2012Metric, symbol dpaa:10u_2
- added C101: 1000u, CP_Radial_D10.0mm_P5.00mm, symbol dpaa:1000u_2
- added C102: 10u, C_0805_2012Metric, symbol dpaa:10u_2
- added C301: 100n, C_0603_1608Metric, symbol dpaa:100n_2
- added C306: 1n 2kV, C_1812_4532Metric, symbol dpaa:1n_2kV_2
- added J19: IDC 2x15, IDC-Header_2x15_P2.54mm_Vertical, symbol dpaa:IDC_2x15_30
- added J29: RB1-125B8G1A, RJ45_UDE_RB1-125B8G1A, symbol dpaa:RB1-125B8G1A_15
- added R301: 0R DNP, R_0603_1608Metric, symbol dpaa:0R_DNP_2
- added R306: 1M, R_0603_1608Metric, symbol dpaa:1M_2
Connections:
- net +5V: now also D1.1 (K), C101.1, C102.1; no longer D1.2 (A)
- net 3V3L: now also R301.2
- net BCLK: now also J20.12; no longer J20.25
- net BTN_TEST: now also J21.10; no longer J21.26
- net CAL: now also J21.12; no longer J21.25
- net ESP_RX: now also J21.8; no longer J21.27
- net ESP_TX: now also J21.6; no longer J21.28
- net GND: now also D1.2 (A), J20.15, J20.21, J20.22, J20.3, J20.4, J21.15, J21.21, J21.22, J21.3, J21.4, C101.2, C102.2, C301.2, C306.1, J19.10, J19.15, J19.16, J19.21, J19.22, J19.27, J19.28, J19.9, R306.2; no longer D1.1 (K), J20.11, J20.2, J20.20, J20.29, J20.8, J21.11, J21.2, J21.20, J21.29, J21.8
- net LRCLK: now also J20.10; no longer J20.26
- net MIC0: now also J21.5; no longer J21.3
- net MIC1: now also J21.7; no longer J21.4
- net MIC10: now also J21.30; no longer J21.16
- net MIC11: now also J21.28; no longer J21.17
- net MIC12: now also J21.26; no longer J21.18
- net MIC13: now also J21.24; no longer J21.19
- net MIC14: now also J21.18; no longer J21.22
- net MIC15: now also J21.14; no longer J21.24
- net MIC2: now also J21.9; no longer J21.5
- net MIC3: now also J21.11; no longer J21.6
- net MIC4: now also J21.13; no longer J21.7
- net MIC5: now also J21.17; no longer J21.9
- net MIC6: now also J21.23; no longer J21.12
- net MIC7: now also J21.25; no longer J21.13
- net MIC8: now also J21.27; no longer J21.14
- net MIC9: now also J21.29; no longer J21.15
- net MON_SD: now also J20.8; no longer J20.27
- net TXD0: now also J20.5; no longer J20.3
- net TXD1: now also J20.7; no longer J20.4
- net TXD10: now also J20.30; no longer J20.16
- net TXD11: now also J20.28; no longer J20.17
- net TXD12: now also J20.26; no longer J20.18
- net TXD13: now also J20.24; no longer J20.19
- net TXD14: now also J20.18; no longer J20.22
- net TXD15: now also J20.14; no longer J20.24
- net TXD2: now also J20.9; no longer J20.5
- net TXD3: now also J20.11; no longer J20.6
- net TXD4: now also J20.13; no longer J20.7
- net TXD5: now also J20.17; no longer J20.9
- net TXD6: now also J20.23; no longer J20.12
- net TXD7: now also J20.25; no longer J20.13
- net TXD8: now also J20.27; no longer J20.14
- net TXD9: now also J20.29; no longer J20.15
- new net CHASSIS: C306.2, J29.R10 (BS GND), J29.SH (SHIELD), R306.1
- new net ETH1_1N: J19.5, J29.R3 (TD1-)
- new net ETH1_1P: J19.7, J29.R2 (TD1+)
- new net ETH1_2N: J19.3, J29.R4 (TD2+)
- new net ETH1_2P: J19.1, J29.R5 (TD2-)
- new net ETH1_3N: J19.6, J29.R7 (TD3-)
- new net ETH1_3P: J19.8, J29.R6 (TD3+)
- new net ETH1_4N: J19.4, J29.R8 (TD4+)
- new net ETH1_4P: J19.2, J29.R9 (TD4-)
- new net ETH_CT: C301.1, J29.R1 (CT), R301.1
- no-connect marks 15 -> 33
